File: hardware/hall-effect-v2.kicad_pcb (KiCad board)
At the start: 2 copper layers, 15 x 25 mm, 29 parts, among them P1 CON-SENSOR2, P2 BOOT, P3 DEBUG, U1 XMC1XXX24, U2 DRV5053, U3 DRILL, U4 DRILL, U5 DRILL, U6 DRILL

Commit message: changed processor to XMC1100
Parts:
- U1: value XMC1XXX24 -> XMC1100
Changed lines of the file:
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@@
     (pad_drill 0)
     (pad_to_mask_clearance 0)
+    (solder_mask_min_width 0.25)
     (aux_axis_origin 176.9 165.9)
     (grid_origin 176.9 165.9)
@@
       (effects (font (size 0.3 0.3) (thickness 0.075)))
     )
-    (fp_text value XMC1XXX24 (at 0 0.8 225) (layer F.Fab)
+    (fp_text value XMC1100 (at 0 0.8 225) (layer F.Fab)
       (effects (font (size 0.3 0.3) (thickness 0.075)))
     )

Commit message: changed processor to XMC1302
Parts:
- U1: value XMC1100 -> XMC1302
Changed lines of the file:
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@@
       (effects (font (size 0.3 0.3) (thickness 0.075)))
     )
-    (fp_text value XMC1100 (at 0 0.8 225) (layer F.Fab)
+    (fp_text value XMC1302 (at 0 0.8 225) (layer F.Fab)
       (effects (font (size 0.3 0.3) (thickness 0.075)))
     )

Commit message: change rc values for voltage generation
Parts:
- C4, C5: value 100nF -> 1uF
- R1, R2: value 1k -> 10k
Changed lines of the file:
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@@
       (effects (font (size 0.2 0.2) (thickness 0.05)))
     )
-    (fp_text value 100nF (at 0.05 -0.375) (layer F.Fab)
+    (fp_text value 1uF (at 0.05 -0.375) (layer F.Fab)
       (effects (font (size 0.2 0.2) (thickness 0.05)))
     )
@@
       (effects (font (size 0.2 0.2) (thickness 0.05)))
     )
-    (fp_text value 100nF (at 0.05 -0.375) (layer F.Fab)
+    (fp_text value 1uF (at 0.05 -0.375) (layer F.Fab)
       (effects (font (size 0.2 0.2) (thickness 0.05)))
     )
@@
       (effects (font (size 0.2 0.2) (thickness 0.05)))
     )
-    (fp_text value 1k (at 0.05 -0.375) (layer F.Fab)
+    (fp_text value 10k (at 0.05 -0.375) (layer F.Fab)
       (effects (font (size 0.2 0.2) (thickness 0.05)))
     )
@@
       (effects (font (size 0.2 0.2) (thickness 0.05)))
     )
-    (fp_text value 1k (at 0.05 -0.375) (layer F.Fab)
-      (effects (font (size 0.2 0.2) (thickness 0.05)))
-    )
+    (fp_text value 10k (at 0.05 -0.375) (layer F.Fab)
+      (effects (font (size 0.2 0.2) (thickness 0.05)))
+    )
